File: FatChudRuns/POWER.kicad_sch (KiCad schematic)
At the start: 17 parts, among them J4 TYPE-C-31-M-12, U3 USBLC6-2SC6, U4 ST730M33R, U6 ST730M33R

Commit message: added 4pF caps and Rext to XTAL, initial placement of PCB, added board outline and gnd plane
Parts:
- U4, U6: footprint SOT_30M33R_STM:SOT_30M33R_STM -> SOT_30M33R_STM
Other:
- moved on the sheet: R53
Changed lines of the file:
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@@
 	)
 	(junction
-		(at 172.72 129.54)
-		(diameter 0)
-		(color 0 0 0 0)
-	)
-	(junction
-		(at 172.72 161.29)
+		(at 176.53 161.29)
 		(diameter 0)
 		(color 0 0 0 0)
@@
 	)
 	(junction
+		(at 176.53 129.54)
+		(diameter 0)
+		(color 0 0 0 0)
+	)
+	(junction
 		(at 91.44 101.6)
 		(diameter 0)
@@
 	(wire
 		(pts
-			(xy 140.97 101.6) (xy 172.72 101.6)
+			(xy 140.97 101.6) (xy 176.53 101.6)
 		)
 		(stroke
@@
 	(wire
 		(pts
+			(xy 176.53 129.54) (xy 187.96 129.54)
+		)
+		(stroke
+			(width 0)
+			(type default)
+		)
+	)
+	(wire
+		(pts
 			(xy 102.87 101.6) (xy 100.33 101.6)
 		)
@@
 	(wire
 		(pts
-			(xy 161.29 161.29) (xy 172.72 161.29)
+			(xy 167.64 161.29) (xy 176.53 161.29)
 		)
 		(stroke
@@
 	(wire
 		(pts
-			(xy 172.72 101.6) (xy 172.72 110.49)
+			(xy 176.53 101.6) (xy 176.53 110.49)
 		)
 		(stroke
@@
 	(wire
 		(pts
+			(xy 176.53 161.29) (xy 187.96 161.29)
+		)
+		(stroke
+			(width 0)
+			(type default)
+		)
+	)
+	(wire
+		(pts
 			(xy 147.32 156.21) (xy 187.96 156.21)
 		)
@@
 	(wire
 		(pts
-			(xy 172.72 129.54) (xy 172.72 161.29)
+			(xy 176.53 129.54) (xy 176.53 161.29)
 		)
 		(stroke
@@
 	(wire
 		(pts
-			(xy 172.72 118.11) (xy 172.72 129.54)
+			(xy 176.53 118.11) (xy 176.53 129.54)
 		)
 		(stroke
@@
 	(wire
 		(pts
-			(xy 172.72 129.54) (xy 187.96 129.54)
-		)
-		(stroke
-			(width 0)
-			(type default)
-		)
-	)
-	(wire
-		(pts
 			(xy 100.33 101.6) (xy 100.33 111.76)
 		)
@@
 	(wire
 		(pts
-			(xy 172.72 161.29) (xy 187.96 161.29)
-		)
-		(stroke
-			(width 0)
-			(type default)
-		)
-	)
-	(wire
-		(pts
 			(xy 203.2 207.01) (xy 203.2 209.55)
 		)
@@
 		)
 	)
-	(label "LDO_EN"
-		(at 161.29 161.29 0)
+	(label "+3.3V"
+		(at 227.33 124.46 0)
+		(effects
+			(font
+				(size 1.27 1.27)
+			)
+			(justify left bottom)
+		)
+	)
+	(label "+3.3VA"
+		(at 227.33 156.21 0)
+		(effects
+			(font
+				(size 1.27 1.27)
+			)
+			(justify left bottom)
+		)
+	)
+	(label "GND"
+		(at 63.5 143.51 0)
+		(effects
+			(font
+				(size 1.27 1.27)
+			)
+			(justify left bottom)
+		)
+	)
+	(label "+5V"
+		(at 115.57 101.6 0)
 		(effects
 			(font
@@
 		)
 	)
+	(global_label "LDO_EN"
+		(shape input)
+		(at 167.64 161.29 180)
+		(fields_autoplaced yes)
+		(effects
+			(font
+				(size 1.27 1.27)
+			)
+			(justify right)
+		)
+		(property "Intersheetrefs" "${INTERSHEET_REFS}"
+			(at 157.484 161.29 0)
+			(effects
+				(font
+					(size 1.27 1.27)
+				)
+				(justify right)
+				(hide yes)
+			)
+		)
+	)
 	(global_label "USB_D-"
 		(shape bidirectional)
@@
 	(symbol
 		(lib_id "Device:R")
-		(at 172.72 114.3 0)
+		(at 176.53 114.3 0)
 		(unit 1)
 		(exclude_from_sim no)
@@
 		(fields_autoplaced yes)
 		(property "Reference" "R53"
-			(at 175.26 113.0299 0)
+			(at 179.07 113.0299 0)
 			(effects
 				(font
@@
 		)
 		(property "Value" "4.7k"
-			(at 175.26 115.5699 0)
+			(at 179.07 115.5699 0)
 			(effects
 				(font
@@
 		)
 		(property "Footprint" "Resistor_SMD:R_0603_1608Metric"
-			(at 170.942 114.3 90)
+			(at 174.752 114.3 90)
 			(effects
 				(font
@@
 		)
 		(property "Datasheet" "~"
-			(at 172.72 114.3 0)
+			(at 176.53 114.3 0)
 			(effects
 				(font
@@
 		)
 		(property "Description" "Resistor"
-			(at 172.72 114.3 0)
+			(at 176.53 114.3 0)
 			(effects
 				(font
@@
 			)
 		)
-		(property "Footprint" "SOT_30M33R_STM:SOT_30M33R_STM"
+		(property "Footprint" "SOT_30M33R_STM"
 			(at 177.8 157.48 0)
 			(effects
@@
 	)
 	(symbol
-		(lib_name "ST730M33R_1")
 		(lib_id "ST730:ST730M33R")
 		(at 177.8 125.73 0)
@@
 			)
 		)
-		(property "Footprint" "SOT_30M33R_STM:SOT_30M33R_STM"
+		(property "Footprint" "SOT_30M33R_STM"
 			(at 177.8 125.73 0)
 			(effects
