File: FatChudRuns/POWER.kicad_sch (KiCad schematic)
At the start: 17 parts, among them J4 TYPE-C-31-M-12, U3 USBLC6-2SC6, U4 ST730M33R, U6 ST730M33R

Commit message: routed phy usb and clock
Parts:
- U4, U6: footprint SOT_30M33R_STM -> SOT_30M33R_STM:SOT_30M33R_STM

Commit message: updated 10uF to 0805, completed BOM, sent to fab
Parts:
- C21, C22, C23, C24: JLCPCB Part # (none) -> C561804; Manufacturer Number (none) -> C0603C105K4PACAUTO
- D1, D2: JLCPCB Part # (none) -> C73929; Manufacturer Number (none) -> IR26-21C/L110/TR8
- J4: JLCPCB Part # (none) -> C165948; Manufacturer Number (none) -> TYPE-C-31-M-12
- R47, R48: JLCPCB Part # (none) -> C14677; Manufacturer Number (none) -> RC0603JR-075K1L
- R49, R54: JLCPCB Part # (none) -> C95177; Manufacturer Number (none) -> RC0603JR-070RL
- R50, R51: JLCPCB Part # (none) -> C107696; Manufacturer Number (none) -> RC0603FR-07220RL
- R53: JLCPCB Part # (none) -> C99782; Manufacturer Number (none) -> RC0603FR-074K7L
- U3: JLCPCB Part # (none) -> C7519; Manufacturer Number (none) -> USBLC6-2SC6
- U4, U6: JLCPCB Part # (none) -> C2846046; Manufacturer Number (none) -> ST730M33R
